File: catProject.kicad_pcb (KiCad board)
At the start: 2 copper layers, 75 x 45 mm, 33 parts, among them IC1 ESP32-S3-WROOM-1-N16R8, J1 USB_C_Receptacle_USB2.0_14P, J3 Conn_01x02, J4 Conn_01x24, U1 TP4056-42-ESOP8, U3 USBLC6-2SC6

Commit message: updated pcb
Parts:
- added Servo3: Conn_01x03, Connector_PinHeader_2.54mm:PinHeader_1x03_P2.54mm_Vertical, F.Cu at (205.2, 70.3)
Connections:
- IC1 pad 18: unconnected-(IC1-IO10-Pad18) -> /SERVO3
Routing:
- net /SERVO3: track 0.00 -> 64.6 mm, vias 0 -> 4
- net +5V: track 90.4 -> 98.9 mm

Commit message: updated PCB, FPC n Servos
Parts:
- added RCAP1: 100nF, Resistor_SMD:R_0805_2012Metric, F.Cu at (159.1, 74.0)
- added RCAP2: 100nF, Resistor_SMD:R_0805_2012Metric, F.Cu at (153.7, 74.0)
Connections:
- J4 pad 1: +3V3 -> unconnected-(J4-Pin_1-Pad1)
- J4 pad 10: /CAM_D6 -> /CAP2
- J4 pad 11: /CAM_D5 -> +3V3
- J4 pad 12: /CAM_D4 -> /CAM_D7
- J4 pad 13: /CAM_D3 -> /CAM_XCLK
- J4 pad 14: /CAM_D2 -> /CAM_D6
- J4 pad 15: /CAM_D1 -> GND
- J4 pad 16: /CAM_D0 -> /CAM_D5
- J4 pad 17: /CAM_RESET -> /CAM_PCLK
- J4 pad 18: /CAM_PWDN -> /CAM_D4
- J4 pad 19: GND -> /CAM_D0
- J4 pad 20: GND -> /CAM_D3
- J4 pad 21: GND -> /CAM_D1
- J4 pad 22: GND -> /CAM_D2
- J4 pad 23: GND -> unconnected-(J4-Pin_23-Pad23)
- J4 pad 24: GND -> unconnected-(J4-Pin_24-Pad24)
- J4 pad 3: /CAM_SIOC -> /CAM_SIOD
- J4 pad 4: /CAM_SIOD -> /CAP1
- J4 pad 5: /CAM_VSYNC -> /CAM_SIOC
- J4 pad 6: /CAM_HREF -> /CAM_RESET
- J4 pad 7: /CAM_PCLK -> /CAM_VSYNC
- J4 pad 8: /CAM_XCLK -> /CAM_PWDN
- J4 pad 9: /CAM_D7 -> /CAM_HREF
Routing:
- net GND: track 137.3 -> 178.4 mm, vias 10 -> 13
- net /CAM_D7: track 19.0 -> 57.4 mm
- net /CAM_SIOD: track 108.9 -> 79.5 mm, vias 5 -> 6
- net /CAM_D3: track 48.5 -> 27.4 mm, vias 2 -> 4
- net /CAM_D2: track 40.4 -> 27.0 mm, vias 2 -> 4
- net /CAM_VSYNC: track 42.3 -> 29.5 mm, vias 4 -> 2
- net /CAP2: track 0.00 -> 12.0 mm, vias 0 -> 2
- net /CAM_D1: track 37.2 -> 26.7 mm, vias 2 -> 4
- net /CAM_XCLK: track 59.0 -> 68.4 mm, vias 2 -> 4
- net /CAM_PCLK: track 37.7 -> 44.6 mm
- net /CAM_D4: track 52.7 -> 45.9 mm
- net /CAM_SIOC: track 76.7 -> 70.6 mm, vias 5 -> 3
- net +3V3: track 140.7 -> 145.8 mm, vias 11 -> 10
- net /CAM_HREF: track 42.9 -> 37.9 mm, vias 4 -> 0
- net /CAM_D0: track 32.9 -> 37.8 mm, vias 0 -> 2
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