File: catProject.kicad_sch (KiCad schematic)
At the start: 30 parts, among them IC1 ESP32-S3-WROOM-1-N16R8, J1 USB_C_Receptacle_USB2.0_14P, J3 Conn_01x02, J4 Conn_01x24, U1 TP4056-42-ESOP8, U3 USBLC6-2SC6

Commit message: updated PCB, FPC n Servos
Parts:
- removed BATT_CONNECT2: Conn_01x02, Connector_PinHeader_2.54mm:PinHeader_1x02_P2.54mm_Vertical, symbol Connector_Generic:Conn_01x02
- added RCAP1, RCAP2: 100nF, Resistor_SMD:R_0805_2012Metric, symbol Device:R
- added Servo3: Conn_01x03, Connector_PinHeader_2.54mm:PinHeader_1x03_P2.54mm_Vertical, symbol Connector_Generic:Conn_01x03
Connections:
- net +3V3: now also J4.11 (Pin_11); no longer J4.1 (Pin_1)
- net +5V: now also Servo3.2 (Pin_2)
- net CAM_D0: now also J4.19 (Pin_19); no longer J4.16 (Pin_16)
- net CAM_D1: now also J4.21 (Pin_21); no longer J4.15 (Pin_15)
- net CAM_D2: now also J4.22 (Pin_22); no longer J4.14 (Pin_14)
- net CAM_D3: now also J4.20 (Pin_20); no longer J4.13 (Pin_13)
- net CAM_D4: now also J4.18 (Pin_18); no longer J4.12 (Pin_12)
- net CAM_D5: now also J4.16 (Pin_16); no longer J4.11 (Pin_11)
- net CAM_D6: now also J4.14 (Pin_14); no longer J4.10 (Pin_10)
- net CAM_D7: now also J4.12 (Pin_12); no longer J4.9 (Pin_9)
- net CAM_HREF: now also J4.9 (Pin_9); no longer J4.6 (Pin_6)
- net CAM_PCLK: now also J4.17 (Pin_17); no longer J4.7 (Pin_7)
- net CAM_PWDN: now also J4.8 (Pin_8); no longer J4.18 (Pin_18)
- net CAM_RESET: now also J4.6 (Pin_6); no longer J4.17 (Pin_17)
- net CAM_SIOC: now also J4.5 (Pin_5); no longer J4.3 (Pin_3)
- net CAM_SIOD: now also J4.3 (Pin_3); no longer J4.4 (Pin_4)
- net CAM_VSYNC: now also J4.7 (Pin_7); no longer J4.5 (Pin_5)
- net CAM_XCLK: now also J4.13 (Pin_13); no longer J4.8 (Pin_8)
- net GND: now also J4.15 (Pin_15), RCAP1.2, RCAP2.2, Servo3.3 (Pin_3); no longer J4.19 (Pin_19), J4.20 (Pin_20), J4.21 (Pin_21), J4.22 (Pin_22), J4.23 (Pin_23), J4.24 (Pin_24)
- net SERVO3: now reaches IC1.18 (IO10)
- net SERVO3: now also Servo3.1 (Pin_1)
- new net CAP1: J4.4 (Pin_4), RCAP1.1
- new net CAP2: J4.10 (Pin_10), RCAP2.1
- no-connect marks 20 -> 22
Other:
- moved on the sheet: CAM_SIOD_R1, ENtiming1, ModuleFast1
